Commit message: ik fixed

File: gym_envs/models/ur5e_gripper/ur5e_gripper.urdf (robot description, URDF)
Before this commit: robot ur5e, 9 links, 8 joints
Joints:
- joint wrist_3_link-tool0_fixed_joint: origin xyz=0 0.34 0 rpy=-1.57079632679 0 -1.57079632679  -> xyz=0 0.1 0 rpy=-1.57079632679 0 -1.57079632679 

Commit message: general update

File: gym_envs/models/ur5e_gripper/ur5e_gripper.urdf (robot description, URDF)
Before this commit: robot ur5e, 9 links, 8 joints
Joints:
- joint wrist_3_link-tool0_fixed_joint: origin xyz=0 0.1 0 rpy=-1.57079632679 0 -1.57079632679  -> xyz=0 0.1 0 rpy=1.57079632679 0 0
