Commit message: update envs

File: gym_envs/models/ur3_robot.urdf (robot description, URDF)
Before this commit: robot ur3, 11 links, 10 joints
Links:
- removed link base
- removed link forearm_link
- removed link world
- link base_link: mass 2.0 -> None; geometry 
- link ee_link: geometry 
- link shoulder_link: mass 2.0 -> None; geometry 
- link upper_arm_link: mass 3.42 -> None; geometry 
- link wrist_1_link: mass 0.8 -> None; geometry 
- link wrist_2_link: mass 0.8 -> None; geometry 
- link wrist_3_link: mass 0.35 -> None; geometry 
Joints:
- removed joint base_link-base_fixed_joint
- removed joint world_joint
- removed joint wrist_3_link-tool0_fixed_joint
- joint ee_fixed_joint: child ee_link -> tool0; origin xyz=0.0 0.0819 0.0 rpy=0.0 0.0 1.570796325 -> xyz=0.0 0.0819 0.0 rpy=-1.5707963 0.0 1.570796325; parent wrist_3_link -> ee_link
- joint elbow_joint: child forearm_link -> wrist_1_link; limit lower=-3.14159265 upper=3.14159265 effort=150.0 velocity=3.15 -> (none)
- joint shoulder_lift_joint: limit lower=-6.2831853 upper=6.2831853 effort=330.0 velocity=2.16 -> (none)
- joint shoulder_pan_joint: limit lower=-6.2831853 upper=6.2831853 effort=330.0 velocity=2.16 -> (none); origin xyz=0.0 0.0 0.1519 rpy=0.0 0.0 0.0 -> xyz=0.0 0.0 1.023 rpy=0.0 0.0 0.0
- joint wrist_1_joint: child wrist_1_link -> wrist_2_link; limit lower=-6.2831853 upper=6.2831853 effort=54.0 velocity=3.2 -> (none); parent forearm_link -> wrist_1_link
- joint wrist_2_joint: child wrist_2_link -> wrist_3_link; limit lower=-6.2831853 upper=6.2831853 effort=54.0 velocity=3.2 -> (none); parent wrist_1_link -> wrist_2_link
- joint wrist_3_joint: child wrist_3_link -> ee_link; limit lower=-6.2831853 upper=6.2831853 effort=54.0 velocity=3.2 -> (none); parent wrist_2_link -> wrist_3_link

Commit message: kdl_ik + correct finger joint

File: gym_envs/models/ur3_robot.urdf (robot description, URDF)
Before this commit: robot ur3, 8 links, 7 joints
Joints:
- joint ee_fixed_joint: origin xyz=0.0 0.0819 0.0 rpy=-1.5707963 0.0 1.570796325 -> xyz=0.0 0.0819 0.0 rpy=-1.5707963 0.0 0
- joint shoulder_pan_joint: origin xyz=0.0 0.0 1.023 rpy=0.0 0.0 0.0 -> xyz=0.0 0.0 1.003 rpy=0.0 0.0 0.0

Commit message: mujoco2.3.0

File: gym_envs/models/ur3_robot.urdf (robot description, URDF)
Before this commit: robot ur3, 8 links, 7 joints
Joints:
- joint ee_fixed_joint: origin xyz=0.0 0.0819 0.0 rpy=-1.5707963 0.0 0 -> xyz=0.0 0.2619 0.0 rpy=-1.5707963 0.0 0
- joint shoulder_pan_joint: origin xyz=0.0 0.0 1.003 rpy=0.0 0.0 0.0 -> xyz=0.0 0.0 1.013 rpy=0.0 0.0 0.0

Commit message: general update

File: gym_envs/models/ur3_robot.urdf (robot description, URDF)
Before this commit: robot ur3, 8 links, 7 joints
Links:
- added link forearm_link
Joints:
- added joint wrist_3_link-tool0_fixed_joint: type fixed, parent wrist_3_link, child tool0, origin xyz=0 0.1 0 rpy=1.57079632679 0 0
- joint ee_fixed_joint: child tool0 -> ee_link; origin xyz=0.0 0.2619 0.0 rpy=-1.5707963 0.0 0 -> xyz=0.0 0.1 0.0 rpy=0.0 0.0 1.57079632679; parent ee_link -> wrist_3_link
- joint elbow_joint: child wrist_1_link -> forearm_link
- joint shoulder_pan_joint: origin xyz=0.0 0.0 1.013 rpy=0.0 0.0 0.0 -> xyz=0.0 0.0 1.023 rpy=0.0 0.0 0.0
- joint wrist_1_joint: child wrist_2_link -> wrist_1_link; parent wrist_1_link -> forearm_link
- joint wrist_2_joint: child wrist_3_link -> wrist_2_link; parent wrist_2_link -> wrist_1_link
- joint wrist_3_joint: child ee_link -> wrist_3_link; parent wrist_3_link -> wrist_2_link

File: gym_envs/models/ur5e_gripper/ur5e_gripper_real.urdf (robot description, URDF)
Before this commit: robot ur5e, 9 links, 8 joints
Joints:
- joint shoulder_pan_joint: origin xyz=0.0 0.0 0.163 rpy=0.0 0.0 0.0 -> xyz=0.0 0.0 0.163 rpy=0.0 0.0 3.14
- joint wrist_3_link-tool0_fixed_joint: origin xyz=0 0.1 0 rpy=1.57079632679 0 0 -> xyz=0 0.28 0 rpy=1.57079632679 0 0

Commit message: upgrade the run.py and envs

File: gym_envs/models/ur3_robot.urdf (robot description, URDF)
Before this commit: robot ur3, 9 links, 8 joints
Joints:
- joint shoulder_pan_joint: origin xyz=0.0 0.0 1.023 rpy=0.0 0.0 0.0 -> xyz=0.0 0.0 1.023 rpy=0.0 0.0 3.14
- joint wrist_3_link-tool0_fixed_joint: origin xyz=0 0.1 0 rpy=1.57079632679 0 0 -> xyz=0 0.26808 0 rpy=1.57079632679 0 0

File: gym_envs/models/ur3_robot_real.urdf (robot description, URDF)
Before this commit: robot ur3, 8 links, 7 joints
Links:
- removed link ee_link
- added link forearm_link
Joints:
- removed joint ee_fixed_joint
- added joint wrist_3_link-tool0_fixed_joint: type fixed, parent wrist_3_link, child tool0, origin xyz=0 0.26808 0 rpy=1.5707 0 0
- joint elbow_joint: child wrist_1_link -> forearm_link
- joint shoulder_lift_joint: origin xyz=0.0 0.1378 0.0 rpy=0.0 1.570796325 0.0 -> xyz=-0.0015 0.1198 0.0 rpy=0.0 1.570796325 0.0
- joint shoulder_pan_joint: origin xyz=0.0 0.0 1 rpy=0.0 0.0 0.0 -> xyz=0.0 0.0 0.153 rpy=0.0 0.0 3.14
- joint wrist_1_joint: child wrist_2_link -> wrist_1_link; origin xyz=0.0 0.0 0.21325 rpy=0.0 1.570796325 0.0 -> xyz=0.0 0.02075 0.21325 rpy=0.0 1.570796325 0.0; parent wrist_1_link -> forearm_link
- joint wrist_2_joint: child wrist_3_link -> wrist_2_link; parent wrist_2_link -> wrist_1_link
- joint wrist_3_joint: child ee_link -> wrist_3_link; parent wrist_3_link -> wrist_2_link
